File: hw/schematic/power-cube.kicad_pcb (KiCad board)
At the start: 2 copper layers, 200 x 50 mm, 50 parts, among them J1 Conn_01x03, J2 Conn_01x04, M1 INA226-MOD, M2 HUSB238-USBPD, M3 USBC-MOD, M4 WEACT-STM32G474, M5 BlueM-D100, M6 BMP280-MOD, Q1 IRF7404, Q2 IRF7404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

Commit message: mod schematic
Parts:
- removed REF**: D_0805_2012Metric_Pad1.15x1.40mm_HandSolder, Diode_SMD:D_0805_2012Metric_Pad1.15x1.40mm_HandSolder
- added D6: SS34, Diode_SMD:D_SMA, F.Cu at (113.7, 24.2)
- C3: value N.M. -> 1000pF
- C5: value 1uF -> 1000pF
- C7: value 0.1uF -> 1uF
- C8: value 1uF -> 10uF
- L1: footprint Capacitor_THT:C_Axial_L3.8mm_D2.6mm_P10.00mm_Horizontal -> Inductor_THT:L_Axial_L5.3mm_D2.2mm_P10.16mm_Horizontal_Vishay_IM-1
- R1, R10: value 200K -> 47K
- R12, R4: value 40K -> 10K
- R14, R7: value 200R -> 330R
- R16: value 100K -> 200K
- R2, R3: value N.M. -> 1K
- R6: footprint Resistor_SMD:R_0603_1608Metric_Pad0.98x0.95mm_HandSolder -> Resistor_SMD:R_0805_2012Metric_Pad1.20x1.40mm_HandSolder
- R8: value 40K -> 40.2K; footprint Resistor_SMD:R_0603_1608Metric_Pad0.98x0.95mm_HandSolder -> Resistor_SMD:R_0805_2012Metric_Pad1.20x1.40mm_HandSolder
- moved R6 59.9 mm to (106.3, 19.7), turned to 180 degrees
- moved R8 57.1 mm to (104.5, 22.2), turned to 180 degrees
- moved U1 12.7 mm to (101.0, 22.2), turned to 0 degrees
- moved R7 10.2 mm to (187.3, 49.1)
- moved C8 7.64 mm to (103.5, 28.8), turned to -90 degrees
- moved C4 6.12 mm to (199.6, 50.1), turned to 0 degrees
- moved C9 5.55 mm to (106.1, 28.8), turned to -90 degrees
- moved R9 5.08 mm to (184.8, 49.1)
- moved C1 2.62 mm to (199.6, 55.2)
- moved R12 1.81 mm to (199.8, 40.0)
- moved R10 1.37 mm to (198.8, 43.5)
Connections:
- C1 pad 1: Net-(Q1-G) -> GND
- C4 pad 1: Net-(Q4-G) -> GND
- C5 pad 2: VDD -> VDC
- D2 pad 2: VCC -> +3V3
- Q4 pad 5: VDD -> VDC
- Q4 pad 6: VDD -> VDC
- Q4 pad 7: VDD -> VDC
- Q4 pad 8: VDD -> VDC
- R2 pad 1: VCC -> +3V3
- R3 pad 1: VCC -> +3V3
- R6 pad 1: VDD -> VDC
Routing:
- net VDC: track 0.00 -> 61.3 mm, vias 0 -> 5
- net VCC: track 130.0 -> 69.7 mm, vias 3 -> 0
- net +3V3: track 64.3 -> 122.6 mm, vias 2 -> 4
- net VDD: track 145.7 -> 104.0 mm, vias 4 -> 3
- net BLUETOOTH_RST: track 5.61 -> 29.3 mm
- net VBUS_ADC: track 44.4 -> 28.3 mm
- net /VBUS_OUT0: track 77.0 -> 64.3 mm
- net VBUS_POWER: track 38.6 -> 49.9 mm, vias 3 -> 4
- net Net-(Q1-G): track 32.4 -> 21.8 mm, vias 0 -> 2
- net EN_EXTRAPWR: track 16.8 -> 22.9 mm
- net GND: track 366.9 -> 362.1 mm, vias 13 -> 9
- net Net-(Q4-G): track 11.9 -> 8.09 mm
- net I2C2_SDA: track 6.35 -> 9.30 mm
- net Net-(J2-Pin_1): track 2.54 -> 0.00 mm
- net VBUS: track 40.4 -> 41.9 mm
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